File: kc65alps.sch (KiCad schematic (older format))
At the start: 14 parts

Commit message: Schematic update
Parts:
- removed SW?: SW_Push, symbol Switch:SW_Push
- added J?: AVR-ISP-6, symbol Connector:AVR-ISP-6
Connections:
- net labels added: MISO, MOSI, RST, SCK
- wire segments 41 -> 48
Changed lines of the file:
@@
 EESchema Schematic File Version 4
+LIBS:kc65alps-cache
 EELAYER 30 0
 EELAYER END
@@
 	1250 2150 1250 2250
 $Comp
-L Switch:SW_Push SW?
-U 1 1 5DF9B2B6
-P 1550 1500
-F 0 "SW?" H 1550 1785 50  0000 C CNN
-F 1 "SW_Push" H 1550 1694 50  0000 C CNN
-F 2 "" H 1550 1700 50  0001 C CNN
-F 3 "~" H 1550 1700 50  0001 C CNN
-	1    1550 1500
-	1    0    0    -1
-$EndComp
-$Comp
-L power:GND #PWR?
-U 1 1 5DF9C33C
-P 1200 1500
-F 0 "#PWR?" H 1200 1250 50  0001 C CNN
-F 1 "GND" H 1205 1327 50  0000 C CNN
-F 2 "" H 1200 1500 50  0001 C CNN
-F 3 "" H 1200 1500 50  0001 C CNN
-	1    1200 1500
-	1    0    0    -1
-$EndComp
-Wire Wire Line
-	1200 1500 1350 1500
-Wire Wire Line
-	1750 1500 1750 1600
-Wire Wire Line
-	1750 1600 1800 1600
-$Comp
 L Device:R_Small R?
 U 1 1 5DF9EA48
@@
 Text GLabel 650  2700 0    50   Input ~ 0
 D-
+$Comp
+L Connector:AVR-ISP-6 J?
+U 1 1 5DF707AD
+P 4600 1750
+F 0 "J?" H 4321 1846 50  0000 R CNN
+F 1 "AVR-ISP-6" H 4321 1755 50  0000 R CNN
+F 2 "" V 4350 1800 50  0001 C CNN
+F 3 " ~" H 3325 1200 50  0001 C CNN
+	1    4600 1750
+	1    0    0    -1
+$EndComp
+$Comp
+L power:+5V #PWR?
+U 1 1 5DF73003
+P 4500 1100
+F 0 "#PWR?" H 4500 950 50  0001 C CNN
+F 1 "+5V" H 4515 1273 50  0000 C CNN
+F 2 "" H 4500 1100 50  0001 C CNN
+F 3 "" H 4500 1100 50  0001 C CNN
+	1    4500 1100
+	1    0    0    -1
+$EndComp
+$Comp
+L power:GND #PWR?
+U 1 1 5DF73F7A
+P 4500 2300
+F 0 "#PWR?" H 4500 2050 50  0001 C CNN
+F 1 "GND" H 4505 2127 50  0000 C CNN
+F 2 "" H 4500 2300 50  0001 C CNN
+F 3 "" H 4500 2300 50  0001 C CNN
+	1    4500 2300
+	1    0    0    -1
+$EndComp
+Text GLabel 5200 1550 2    50   Input ~ 0
+MISO
+Text GLabel 5200 1650 2    50   Input ~ 0
+MOSI
+Text GLabel 5250 1750 2    50   Input ~ 0
+SCK
+Text GLabel 5250 1850 2    50   Input ~ 0
+RST
+Wire Wire Line
+	5000 1550 5200 1550
+Wire Wire Line
+	5200 1650 5000 1650
+Wire Wire Line
+	5000 1750 5250 1750
+Wire Wire Line
+	5250 1850 5000 1850
+Wire Wire Line
+	4500 1250 4500 1100
+Wire Wire Line
+	4500 2150 4500 2300
+Text GLabel 1550 1600 0    50   Input ~ 0
+RST
+Wire Wire Line
+	1550 1600 1800 1600
+Text GLabel 3250 1900 2    50   Input ~ 0
+MISO
+Text GLabel 3250 1800 2    50   Input ~ 0
+MOSI
+Text GLabel 3250 1700 2    50   Input ~ 0
+SCK
+Wire Wire Line
+	3050 1700 3250 1700
+Wire Wire Line
+	3250 1800 3050 1800
+Wire Wire Line
+	3050 1900 3250 1900
 $EndSCHEMATC

Commit message: Schematic Update
Parts:
- added J?: Conn_01x04, symbol Connector_Generic:Conn_01x04
Connections:
- net D+: now also J?.3 (Pin_3)
- net D-: now also J?.2 (Pin_2)
- net GND: now also J?.4 (Pin_4)
- new net VCC: J?.1 (Pin_1)
Changed lines of the file:
@@
 Wire Wire Line
 	3050 1900 3250 1900
+$Comp
+L Connector_Generic:Conn_01x04 J?
+U 1 1 5DF85843
+P 5550 3000
+F 0 "J?" H 5630 2992 50  0000 L CNN
+F 1 "Conn_01x04" H 5630 2901 50  0000 L CNN
+F 2 "" H 5550 3000 50  0001 C CNN
+F 3 "~" H 5550 3000 50  0001 C CNN
+	1    5550 3000
+	1    0    0    -1
+$EndComp
+$Comp
+L power:VCC #PWR?
+U 1 1 5DF868E4
+P 5250 2900
+F 0 "#PWR?" H 5250 2750 50  0001 C CNN
+F 1 "VCC" V 5268 3027 50  0000 L CNN
+F 2 "" H 5250 2900 50  0001 C CNN
+F 3 "" H 5250 2900 50  0001 C CNN
+	1    5250 2900
+	0    -1   -1   0
+$EndComp
+$Comp
+L power:GND #PWR?
+U 1 1 5DF87727
+P 5250 3200
+F 0 "#PWR?" H 5250 2950 50  0001 C CNN
+F 1 "GND" H 5255 3027 50  0000 C CNN
+F 2 "" H 5250 3200 50  0001 C CNN
+F 3 "" H 5250 3200 50  0001 C CNN
+	1    5250 3200
+	1    0    0    -1
+$EndComp
+Text GLabel 5250 3000 0    50   Input ~ 0
+D-
+Text GLabel 5250 3100 0    50   Input ~ 0
+D+
+Wire Wire Line
+	5250 3200 5350 3200
+Wire Wire Line
+	5250 3100 5350 3100
+Wire Wire Line
+	5250 3000 5350 3000
+Wire Wire Line
+	5250 2900 5350 2900
 $EndSCHEMATC

Commit message: Schematic Update
Parts:
- added F?: 500mA, symbol Device:Polyfuse_Small
Connections:
- net +5V: now also F?.2
- net VCC: now also F?.1
Other:
- moved on the sheet: C?, J?, R?, U?, Y?

Commit message: Schematic update
Parts:
- added D?: SOD-123, symbol Device:D_Small
- added MX?: MX-NoLED, symbol MX_Alps_Hybrid:MX-NoLED
Connections:
- new net: D?.2 (A), MX?.2 (ROW)
Other:
- note added: "1"
- note added: "191216"
- note added: "AVR ISP Header"
- note added: "Decoupling Capacitors"
- note added: "JST-SR Connection"
- note added: "KC 65 Alps"
- note added: "MCU"
Changed lines of the file:
@@
 Wire Wire Line
 	3700 3700 4000 3700
+Wire Notes Line
+	600  750  4200 750
+Wire Notes Line
+	4200 750  4200 5300
+Wire Notes Line
+	4200 5300 600  5300
+Wire Notes Line
+	600  5300 600  750
+Wire Notes Line
+	4650 750  6600 750
+Wire Notes Line
+	6600 750  6600 2600
+Wire Notes Line
+	6600 2600 4650 2600
+Wire Notes Line
+	4650 2600 4650 750
+Wire Notes Line
+	6750 750  6750 2200
+Wire Notes Line
+	6750 2200 8500 2200
+Wire Notes Line
+	8500 2200 8500 750
+Wire Notes Line
+	8500 750  6750 750
+Wire Notes Line
+	8750 750  8750 2200
+Wire Notes Line
+	8750 2200 10450 2200
+Wire Notes Line
+	10450 2200 10450 750
+Wire Notes Line
+	10450 750  8750 750
+Text Notes 650  700  0    50   ~ 0
+MCU
+Text Notes 4650 700  0    50   ~ 0
+AVR ISP Header
+Text Notes 6750 700  0    50   ~ 0
+JST-SR Connection
+Text Notes 8750 700  0    50   ~ 0
+Decoupling Capacitors
+Text Notes 7350 7500 0    50   ~ 10
+KC 65 Alps
+Text Notes 8150 7650 0    50   ~ 10
+191216
+Text Notes 10600 7650 0    50   ~ 10
+1
+$Comp
+L MX_Alps_Hybrid:MX-NoLED MX?
+U 1 1 5DF931BD
+P 6600 3450
+F 0 "MX?" H 6633 3673 60  0000 C CNN
+F 1 "MX-NoLED" H 6633 3599 20  0000 C CNN
+F 2 "" H 5975 3425 60  0001 C CNN
+F 3 "" H 5975 3425 60  0001 C CNN
+	1    6600 3450
+	1    0    0    -1
+$EndComp
+$Comp
+L Device:D_Small D?
+U 1 1 5DF95296
+P 6350 3700
+F 0 "D?" H 6350 3800 50  0000 R CNN
+F 1 "SOD-123" H 6800 3800 50  0000 R CNN
+F 2 "" V 6350 3700 50  0001 C CNN
+F 3 "~" V 6350 3700 50  0001 C CNN
+	1    6350 3700
+	0    -1   -1   0
+$EndComp
+Wire Wire Line
+	6350 3600 6550 3600
 $EndSCHEMATC

Commit message: Updating Schematic
Parts:
- added D? (x68): SOD-123, symbol Device:D_Small
- added MX? (x75): MX-NoLED, symbol MX_Alps_Hybrid:MX-NoLED
Connections:
- net COL0: now reaches MX?.1 (COL)
- net COL0: now also MX?.1 (COL), MX?.1 (COL), MX?.1 (COL), MX?.2 (ROW), MX?.2 (ROW), MX?.2 (ROW)
- net ROW0: now reaches D?.1 (K)
- net ROW0: now also D?.1 (K), D?.1 (K), D?.1 (K), D?.1 (K), D?.1 (K), D?.1 (K), D?.1 (K), D?.1 (K), D?.1 (K), D?.1 (K), D?.1 (K), D?.1 (K), D?.1 (K), D?.1 (K), D?.1 (K)
- new net: D?.2 (A), MX?.2 (ROW) (x62)
- new net: D?.2 (A), MX?.1 (COL), MX?.2 (ROW) (x5)
- new net: D?.2 (A), MX?.1 (COL), MX?.1 (COL), MX?.2 (ROW)
- new net COL1: MX?.1 (COL), MX?.1 (COL)
- new net COL10: MX?.1 (COL), MX?.1 (COL), MX?.1 (COL), MX?.1 (COL), MX?.1 (COL)
- new net COL11: MX?.1 (COL), MX?.1 (COL), MX?.1 (COL), MX?.1 (COL), MX?.1 (COL), MX?.2 (ROW)
- new net COL12: MX?.1 (COL), MX?.1 (COL), MX?.1 (COL)
- new net COL13: MX?.1 (COL), MX?.1 (COL), MX?.1 (COL), MX?.1 (COL), MX?.1 (COL)
- new net COL14: MX?.1 (COL), MX?.1 (COL), MX?.1 (COL), MX?.1 (COL), MX?.2 (ROW)
- new net COL15: MX?.1 (COL), MX?.1 (COL), MX?.1 (COL), MX?.1 (COL), MX?.1 (COL)
- new net COL2: MX?.1 (COL), MX?.1 (COL), MX?.1 (COL), MX?.1 (COL), MX?.1 (COL), MX?.2 (ROW)
- new net COL3: MX?.1 (COL), MX?.1 (COL), MX?.1 (COL), MX?.1 (COL), MX?.1 (COL), MX?.2 (ROW)
- new net COL4: MX?.1 (COL), MX?.1 (COL), MX?.1 (COL), MX?.1 (COL)
- new net COL5: MX?.1 (COL), MX?.1 (COL), MX?.1 (COL), MX?.1 (COL)
- new net COL6: MX?.1 (COL), MX?.1 (COL), MX?.1 (COL), MX?.1 (COL), MX?.1 (COL)
- new net COL7: MX?.1 (COL), MX?.1 (COL), MX?.1 (COL), MX?.1 (COL), MX?.1 (COL)
- new net COL8: MX?.1 (COL), MX?.1 (COL), MX?.1 (COL), MX?.1 (COL)
- new net COL9: MX?.1 (COL), MX?.1 (COL), MX?.1 (COL), MX?.1 (COL)
- new net ROW1: D?.1 (K), D?.1 (K), D?.1 (K), D?.1 (K), D?.1 (K), D?.1 (K), D?.1 (K), D?.1 (K), D?.1 (K), D?.1 (K), D?.1 (K), D?.1 (K), D?.1 (K), D?.1 (K), D?.1 (K)
- new net ROW2: D?.1 (K), D?.1 (K), D?.1 (K), D?.1 (K), D?.1 (K), D?.1 (K), D?.1 (K), D?.1 (K), D?.1 (K), D?.1 (K), D?.1 (K), D?.1 (K), D?.1 (K), D?.1 (K)
- new net ROW3: D?.1 (K), D?.1 (K), D?.1 (K), D?.1 (K), D?.1 (K), D?.1 (K), D?.1 (K), D?.1 (K), D?.1 (K), D?.1 (K), D?.1 (K), D?.1 (K), D?.1 (K), D?.1 (K)
- new net ROW4: D?.1 (K), D?.1 (K), D?.1 (K), D?.1 (K), D?.1 (K), D?.1 (K), D?.1 (K), D?.1 (K), D?.1 (K), D?.1 (K)
Other:
- note added: "Key Matrix"
- note removed: "1"
- note removed: "191216"
- note removed: "KC 65 Alps"
- moved on the sheet: C?, D?, F?, J?, MX?

Commit message: Schematic update
Parts:
- gave numbers to parts that had none: 21

Commit message: Schematic update
Parts:
- gave numbers to parts that had none: 55
- renumbered MX-backspace1 to MX-Backspace1, MX-backspace2 to MX-Backspace2, MX-e to MX-E, MX-esc to MX-Esc, MX-pgup to MX-PgUp, MX-q to MX-Q, MX-tab to MX-Tab, MX-w to MX-W

Commit message: Schematic update
Parts:
- removed D?: SOD-123, symbol Device:D_Small
- renumbered MX-Space2 to MX-Space1, MX-Space1 to MX-Space2
Connections:
- net COL0: now also MX-LCtrl2.1 (COL); no longer MX-LCtrl2.2 (ROW)
- net COL11: now also MX-RWin2.1 (COL); no longer MX-RWin2.2 (ROW)
- net COL2: now also MX-LWin2.1 (COL); no longer MX-LWin2.2 (ROW)
- net COL3: now also MX-LAlt2.1 (COL); no longer MX-LAlt2.2 (ROW)
- net COL6: no longer MX-Space2.1 (COL)
- net COL7: now also MX-Space2.1 (COL)
- net at D?.2 (A), MX-LCtrl1.2 (ROW): now also MX-LCtrl2.2 (ROW); no longer MX-LCtrl2.1 (COL)
- net at D?.2 (A), MX-LWin1.2 (ROW): now also MX-LWin2.2 (ROW); no longer MX-LWin2.1 (COL)
- net at D?.2 (A), MX-LAlt1.2 (ROW): now also MX-LAlt2.2 (ROW); no longer MX-LAlt2.1 (COL)
- net at D?.2 (A), MX-Space1.2 (ROW): now also MX-Space2.2 (ROW)
- net at D?.2 (A), MX-RWin1.2 (ROW): now also MX-RWin2.2 (ROW); no longer MX-RWin2.1 (COL)
Other:
- moved on the sheet: MX-LAlt2, MX-LCtrl2, MX-LWin2, MX-RWin2, MX-Space2
Changed lines of the file:
@@
 	7450 8900 7650 8900
 $Comp
-L MX_Alps_Hybrid:MX-NoLED MX-Space2
+L MX_Alps_Hybrid:MX-NoLED MX-Space1
 U 1 1 5E25805F
 P 10300 8750
-F 0 "MX-Space2" H 10333 8973 60  0000 C CNN
+F 0 "MX-Space1" H 10333 8973 60  0000 C CNN
 F 1 "MX-NoLED" H 10333 8899 20  0000 C CNN
 F 2 "" H 9675 8725 60  0001 C CNN
@@
 	6800 9100 7450 9100
 Connection ~ 7450 9100
-Wire Wire Line
-	7450 9100 9400 9100
 Connection ~ 10050 9100
 Wire Wire Line
@@
 Connection ~ 14600 5900
 $Comp
-L MX_Alps_Hybrid:MX-NoLED MX-Space1
+L MX_Alps_Hybrid:MX-NoLED MX-Space2
 U 1 1 5E4E11EB
-P 9650 8750
-F 0 "MX-Space1" H 9683 8973 60  0000 C CNN
-F 1 "MX-NoLED" H 9683 8899 20  0000 C CNN
-F 2 "" H 9025 8725 60  0001 C CNN
-F 3 "" H 9025 8725 60  0001 C CNN
-	1    9650 8750
-	1    0    0    -1
-$EndComp
-$Comp
-L Device:D_Small D?
-U 1 1 5E4E11F1
-P 9400 9000
-F 0 "D?" H 9400 9100 50  0000 R CNN
-F 1 "SOD-123" H 9850 9100 50  0000 R CNN
-F 2 "" V 9400 9000 50  0001 C CNN
-F 3 "~" V 9400 9000 50  0001 C CNN
-	1    9400 9000
-	0    -1   -1   0
-$EndComp
-Wire Wire Line
-	9400 8900 9600 8900
-Connection ~ 9400 9100
-Wire Wire Line
-	9400 9100 10050 9100
-Wire Wire Line
-	9800 7950 9800 8700
-Connection ~ 9800 7950
+P 10300 9350
+F 0 "MX-Space2" H 10333 9573 60  0000 C CNN
+F 1 "MX-NoLED" H 10333 9499 20  0000 C CNN
+F 2 "" H 9675 9325 60  0001 C CNN
+F 3 "" H 9675 9325 60  0001 C CNN
+	1    10300 9350
+	1    0    0    -1
+$EndComp
 $Comp
 L MX_Alps_Hybrid:MX-NoLED MX-RWin2
 U 1 1 5E5224A1
-P 13000 9350
-F 0 "MX-RWin2" H 12872 9295 60  0000 R CNN
-F 1 "MX-NoLED" H 12872 9369 20  0000 R CNN
-F 2 "" H 12375 9325 60  0001 C CNN
-F 3 "" H 12375 9325 60  0001 C CNN
-	1    13000 9350
-	-1   0    0    1
-$EndComp
-Wire Wire Line
-	13050 9200 13050 8700
-Connection ~ 13050 8700
-Wire Wire Line
-	12850 9400 12850 8900
-Connection ~ 12850 8900
+P 12900 9350
+F 0 "MX-RWin2" H 12772 9295 60  0000 R CNN
+F 1 "MX-NoLED" H 12772 9369 20  0000 R CNN
+F 2 "" H 12275 9325 60  0001 C CNN
+F 3 "" H 12275 9325 60  0001 C CNN
+	1    12900 9350
+	1    0    0    -1
+$EndComp
 $Comp
 L MX_Alps_Hybrid:MX-NoLED MX-LAlt2
 U 1 1 5E54FCFF
-P 7800 9350
-F 0 "MX-LAlt2" H 7672 9295 60  0000 R CNN
-F 1 "MX-NoLED" H 7672 9369 20  0000 R CNN
-F 2 "" H 7175 9325 60  0001 C CNN
-F 3 "" H 7175 9325 60  0001 C CNN
-	1    7800 9350
-	-1   0    0    1
+P 7700 9350
+F 0 "MX-LAlt2" H 7572 9295 60  0000 R CNN
+F 1 "MX-NoLED" H 7572 9369 20  0000 R CNN
+F 2 "" H 7075 9325 60  0001 C CNN
+F 3 "" H 7075 9325 60  0001 C CNN
+	1    7700 9350
+	1    0    0    -1
 $EndComp
 $Comp
 L MX_Alps_Hybrid:MX-NoLED MX-LWin2
 U 1 1 5E552419
-P 7150 9350
-F 0 "MX-LWin2" H 7022 9295 60  0000 R CNN
-F 1 "MX-NoLED" H 7022 9369 20  0000 R CNN
-F 2 "" H 6525 9325 60  0001 C CNN
-F 3 "" H 6525 9325 60  0001 C CNN
-	1    7150 9350
-	-1   0    0    1
+P 7050 9350
+F 0 "MX-LWin2" H 6922 9295 60  0000 R CNN
+F 1 "MX-NoLED" H 6922 9369 20  0000 R CNN
+F 2 "" H 6425 9325 60  0001 C CNN
+F 3 "" H 6425 9325 60  0001 C CNN
+	1    7050 9350
+	1    0    0    -1
 $EndComp
 $Comp
 L MX_Alps_Hybrid:MX-NoLED MX-LCtrl2
 U 1 1 5E5538F6
-P 5850 9350
-F 0 "MX-LCtrl2" H 5722 9295 60  0000 R CNN
-F 1 "MX-NoLED" H 5722 9369 20  0000 R CNN
-F 2 "" H 5225 9325 60  0001 C CNN
-F 3 "" H 5225 9325 60  0001 C CNN
-	1    5850 9350
-	-1   0    0    1
-$EndComp
-Wire Wire Line
-	7850 8700 7850 9200
-Connection ~ 7850 8700
-Wire Wire Line
-	7650 8900 7650 9400
-Connection ~ 7650 8900
-Wire Wire Line
-	7200 8700 7200 9200
-Connection ~ 7200 8700
-Wire Wire Line
-	7000 8900 7000 9400
-Connection ~ 7000 8900
-Wire Wire Line
-	5900 8700 5900 9200
-Connection ~ 5900 8700
-Wire Wire Line
-	5700 8900 5700 9400
-Connection ~ 5700 8900
+P 5750 9350
+F 0 "MX-LCtrl2" H 5622 9295 60  0000 R CNN
+F 1 "MX-NoLED" H 5622 9369 20  0000 R CNN
+F 2 "" H 5125 9325 60  0001 C CNN
+F 3 "" H 5125 9325 60  0001 C CNN
+	1    5750 9350
+	1    0    0    -1
+$EndComp
 Text GLabel 5200 6100 0    50   Input ~ 0
 ROW0
@@
 	1    0    0    -1
 $EndComp
+Wire Wire Line
+	7450 9100 10050 9100
+Wire Wire Line
+	10450 8700 10450 9300
+Connection ~ 10450 8700
+Wire Wire Line
+	10250 8900 10250 9500
+Connection ~ 10250 8900
+Wire Wire Line
+	7850 8700 7850 9300
+Connection ~ 7850 8700
+Wire Wire Line
+	7650 8900 7650 9500
+Connection ~ 7650 8900
+Wire Wire Line
+	7200 8700 7200 9300
+Connection ~ 7200 8700
+Wire Wire Line
+	7000 8900 7000 9500
+Connection ~ 7000 8900
+Wire Wire Line
+	5900 8700 5900 9300
+Connection ~ 5900 8700
+Wire Wire Line
+	5700 8900 5700 9500
+Connection ~ 5700 8900
+Wire Wire Line
+	13050 8700 13050 9300
+Connection ~ 13050 8700
+Wire Wire Line
+	12850 8900 12850 9500
+Connection ~ 12850 8900
 $EndSCHEMATC
