File: kc65alps.sch (KiCad schematic (older format))
At the start: 160 parts

Commit message: Schematic update
Parts:
- C1, C2, C3, C4, C5, C6, C7: renamed from C?; footprint (none) -> Capacitors_SMD:C_0805
- D1, D10, D11, D12, D13, D14, D15, D16, D17, D18, D19, D2, D20, D21, D22, D23, D24, D25, D26, D27, D28, D29, D3, D30, D31, D32, D33, D34, D35, D36, D37, D38, D39, D4, D40, D41, D42, D43, D44, D45, D46, D47, D48, D49, D5, D50, D51, D52, D53, D54, D55, D56, D57, D58, D59, D6, D60, D61, D62, D63, D64, D65, D66, D67, D68, D7, D8, D9: renamed from D?; footprint (none) -> Diodes_SMD:D_SOD-123
- F1: renamed from F?; footprint (none) -> Fuse_Holders_and_Fuses:Fuse_SMD1206_Reflow
- MX-'1: renamed from MX-'; footprint (none) -> Alps_Only:ALPS-1U
- MX-,1: renamed from MX-,; footprint (none) -> Alps_Only:ALPS-1U
- MX--1: renamed from MX--; footprint (none) -> Alps_Only:ALPS-1U
- MX-.1: renamed from MX-.; footprint (none) -> Alps_Only:ALPS-1U
- MX-/1: renamed from MX-/; footprint (none) -> Alps_Only:ALPS-1U
- MX-0, MX-1, MX-2, MX-3, MX-4, MX-5, MX-6, MX-7, MX-8, MX-9, MX-Backspace1, MX-Backspace2, MX-Caps1, MX-Caps2, MX-Caps3, MX-LAlt1, MX-LAlt2, MX-LCtrl1, MX-LCtrl2, MX-LWin1, MX-LWin2, MX-RWin1, MX-RWin2, MX-Space1, MX-Space2: footprint (none) -> Alps_Only:ALPS-1U
- MX-;1: renamed from MX-;; footprint (none) -> Alps_Only:ALPS-1U
- MX-=1: renamed from MX-=; footprint (none) -> Alps_Only:ALPS-1U
- MX-A1: renamed from MX-A; footprint (none) -> Alps_Only:ALPS-1U
- MX-B1: renamed from MX-B; footprint (none) -> Alps_Only:ALPS-1U
- MX-C1: renamed from MX-C; footprint (none) -> Alps_Only:ALPS-1U
- MX-D1: renamed from MX-D; footprint (none) -> Alps_Only:ALPS-1U
- MX-DArrow1: renamed from MX-DArrow; footprint (none) -> Alps_Only:ALPS-1U
- MX-E1: renamed from MX-E; footprint (none) -> Alps_Only:ALPS-1U
- MX-Enter1: renamed from MX-Enter; footprint (none) -> Alps_Only:ALPS-1U
- MX-Esc1: renamed from MX-Esc; footprint (none) -> Alps_Only:ALPS-1U
- MX-F1: renamed from MX-F; footprint (none) -> Alps_Only:ALPS-1U
- MX-Fn1: renamed from MX-Fn; footprint (none) -> Alps_Only:ALPS-1U
- MX-G1: renamed from MX-G; footprint (none) -> Alps_Only:ALPS-1U
- MX-H1: renamed from MX-H; footprint (none) -> Alps_Only:ALPS-1U
- MX-I1: renamed from MX-I; footprint (none) -> Alps_Only:ALPS-1U
- MX-J1: renamed from MX-J; footprint (none) -> Alps_Only:ALPS-1U
- MX-K1: renamed from MX-K; footprint (none) -> Alps_Only:ALPS-1U
- MX-L1: renamed from MX-L; footprint (none) -> Alps_Only:ALPS-1U
- MX-LArrow1: renamed from MX-LArrow; footprint (none) -> Alps_Only:ALPS-1U
- MX-LShift1: renamed from MX-LShift; footprint (none) -> Alps_Only:ALPS-1U
- MX-M1: renamed from MX-M; footprint (none) -> Alps_Only:ALPS-1U
- MX-N1: renamed from MX-N; footprint (none) -> Alps_Only:ALPS-1U
- MX-O1: renamed from MX-O; footprint (none) -> Alps_Only:ALPS-1U
- MX-P1: renamed from MX-P; footprint (none) -> Alps_Only:ALPS-1U
- MX-PgDn1: renamed from MX-PgDn; footprint (none) -> Alps_Only:ALPS-1U
- MX-PgUp1: renamed from MX-PgUp; footprint (none) -> Alps_Only:ALPS-1U
- MX-Q1: renamed from MX-Q; footprint (none) -> Alps_Only:ALPS-1U
- MX-R1: renamed from MX-R; footprint (none) -> Alps_Only:ALPS-1U
- MX-RAlt1: renamed from MX-RAlt; footprint (none) -> Alps_Only:ALPS-1U
- MX-RArrow1: renamed from MX-RArrow; footprint (none) -> Alps_Only:ALPS-1U
- MX-RShift1: renamed from MX-RShift; footprint (none) -> Alps_Only:ALPS-1U
- MX-S1: renamed from MX-S; footprint (none) -> Alps_Only:ALPS-1U
- MX-Super1: renamed from MX-Super; footprint (none) -> Alps_Only:ALPS-1U
- MX-T1: renamed from MX-T; footprint (none) -> Alps_Only:ALPS-1U
- MX-Tab1: renamed from MX-Tab; footprint (none) -> Alps_Only:ALPS-1U
- MX-U1: renamed from MX-U; footprint (none) -> Alps_Only:ALPS-1U
- MX-UArrow1: renamed from MX-UArrow; footprint (none) -> Alps_Only:ALPS-1U
- MX-V1: renamed from MX-V; footprint (none) -> Alps_Only:ALPS-1U
- MX-W1: renamed from MX-W; footprint (none) -> Alps_Only:ALPS-1U
- MX-X1: renamed from MX-X; footprint (none) -> Alps_Only:ALPS-1U
- MX-Y1: renamed from MX-Y; footprint (none) -> Alps_Only:ALPS-1U
- MX-Z1: renamed from MX-Z; footprint (none) -> Alps_Only:ALPS-1U
- MX-[1: renamed from MX-[; footprint (none) -> Alps_Only:ALPS-1U
- MX-\1: renamed from MX-\; footprint (none) -> Alps_Only:ALPS-1U
- MX-]1: renamed from MX-]; footprint (none) -> Alps_Only:ALPS-1U
- MX-`1: renamed from MX-`; footprint (none) -> Alps_Only:ALPS-1U
- R1, R2, R3, R4: renamed from R?; footprint (none) -> Resistors_SMD:R_0805
- Y1: renamed from Y?; footprint (none) -> Crystals:Crystal_SMD_3225-4pin_3.2x2.5mm
- gave numbers to parts that had none: 3

Commit message: Schematic Update
Parts:
- J1: footprint (none) -> random-keyboard-parts:JST-SR-4
- J2: footprint (none) -> random-keyboard-parts:Reset_Pretty-Mask
- MX-Backspace2: footprint Alps_Only:ALPS-1U -> Alps_Only:ALPS-2U
- MX-Enter1, MX-LShift1: footprint Alps_Only:ALPS-1U -> Alps_Only:ALPS-2.25U
- MX-LAlt1, MX-LCtrl1, MX-Tab1, MX-\1: footprint Alps_Only:ALPS-1U -> Alps_Only:ALPS-1.5U
- MX-LAlt2, MX-LCtrl2, MX-LWin2, MX-RAlt1, MX-RWin2: footprint Alps_Only:ALPS-1U -> Alps_Only:ALPS-1.25U
- MX-RShift1: footprint Alps_Only:ALPS-1U -> Alps_Only:ALPS-1.75U
- MX-Space1: footprint Alps_Only:ALPS-1U -> Alps_Only:ALPS-7U
- MX-Space2: footprint Alps_Only:ALPS-1U -> Alps_Only:ALPS-6.25U
Connections:
- net D+: now also R2.1, U1.4 (D+)
- net D-: now also R3.1, U1.3 (D-)
Changed lines of the file:
@@
 F 0 "J2" H 6521 3396 50  0000 R CNN
 F 1 "AVR-ISP-6" H 6521 3305 50  0000 R CNN
-F 2 "" V 6550 3350 50  0001 C CNN
+F 2 "random-keyboard-parts:Reset_Pretty-Mask" V 6550 3350 50  0001 C CNN
 F 3 " ~" H 5525 2750 50  0001 C CNN
 	1    6800 3300
@@
 F 0 "J1" H 10330 1792 50  0000 L CNN
 F 1 "Conn_01x04" H 10330 1701 50  0000 L CNN
-F 2 "" H 10250 1800 50  0001 C CNN
+F 2 "random-keyboard-parts:JST-SR-4" H 10250 1800 50  0001 C CNN
 F 3 "~" H 10250 1800 50  0001 C CNN
 	1    10250 1800
@@
 F 0 "MX-\\1" H 14883 6723 60  0000 C CNN
 F 1 "MX-NoLED" H 14883 6649 20  0000 C CNN
-F 2 "Alps_Only:ALPS-1U" H 14225 6475 60  0001 C CNN
+F 2 "Alps_Only:ALPS-1.5U" H 14225 6475 60  0001 C CNN
 F 3 "" H 14225 6475 60  0001 C CNN
 	1    14850 6500
@@
 F 0 "MX-Enter1" H 14233 7473 60  0000 C CNN
 F 1 "MX-NoLED" H 14233 7399 20  0000 C CNN
-F 2 "Alps_Only:ALPS-1U" H 13575 7225 60  0001 C CNN
+F 2 "Alps_Only:ALPS-2.25U" H 13575 7225 60  0001 C CNN
 F 3 "" H 13575 7225 60  0001 C CNN
 	1    14200 7250
@@
 F 0 "MX-LShift1" H 6433 8223 60  0000 C CNN
 F 1 "MX-NoLED" H 6433 8149 20  0000 C CNN
-F 2 "Alps_Only:ALPS-1U" H 5775 7975 60  0001 C CNN
+F 2 "Alps_Only:ALPS-2.25U" H 5775 7975 60  0001 C CNN
 F 3 "" H 5775 7975 60  0001 C CNN
 	1    6400 8000
@@
 F 0 "MX-RShift1" H 14233 8223 60  0000 C CNN
 F 1 "MX-NoLED" H 14233 8149 20  0000 C CNN
-F 2 "Alps_Only:ALPS-1U" H 13575 7975 60  0001 C CNN
+F 2 "Alps_Only:ALPS-1.75U" H 13575 7975 60  0001 C CNN
 F 3 "" H 13575 7975 60  0001 C CNN
 	1    14200 8000
@@
 F 0 "MX-LCtrl1" H 5783 8973 60  0000 C CNN
 F 1 "MX-NoLED" H 5783 8899 20  0000 C CNN
-F 2 "Alps_Only:ALPS-1U" H 5125 8725 60  0001 C CNN
+F 2 "Alps_Only:ALPS-1.5U" H 5125 8725 60  0001 C CNN
 F 3 "" H 5125 8725 60  0001 C CNN
 	1    5750 8750
@@
 F 0 "MX-LAlt1" H 7733 8973 60  0000 C CNN
 F 1 "MX-NoLED" H 7733 8899 20  0000 C CNN
-F 2 "Alps_Only:ALPS-1U" H 7075 8725 60  0001 C CNN
+F 2 "Alps_Only:ALPS-1.5U" H 7075 8725 60  0001 C CNN
 F 3 "" H 7075 8725 60  0001 C CNN
 	1    7700 8750
@@
 F 0 "MX-Space1" H 10333 8973 60  0000 C CNN
 F 1 "MX-NoLED" H 10333 8899 20  0000 C CNN
-F 2 "Alps_Only:ALPS-1U" H 9675 8725 60  0001 C CNN
+F 2 "Alps_Only:ALPS-7U" H 9675 8725 60  0001 C CNN
 F 3 "" H 9675 8725 60  0001 C CNN
 	1    10300 8750
@@
 F 0 "MX-RAlt1" H 12283 8973 60  0000 C CNN
 F 1 "MX-NoLED" H 12283 8899 20  0000 C CNN
-F 2 "Alps_Only:ALPS-1U" H 11625 8725 60  0001 C CNN
+F 2 "Alps_Only:ALPS-1.25U" H 11625 8725 60  0001 C CNN
 F 3 "" H 11625 8725 60  0001 C CNN
 	1    12250 8750
@@
 F 0 "MX-Backspace2" H 14683 5573 60  0000 C CNN
 F 1 "MX-NoLED" H 14683 5499 20  0000 C CNN
-F 2 "Alps_Only:ALPS-1U" H 14025 5325 60  0001 C CNN
+F 2 "Alps_Only:ALPS-2U" H 14025 5325 60  0001 C CNN
 F 3 "" H 14025 5325 60  0001 C CNN
 	1    14650 5350
@@
 F 0 "MX-Space2" H 10333 9573 60  0000 C CNN
 F 1 "MX-NoLED" H 10333 9499 20  0000 C CNN
-F 2 "Alps_Only:ALPS-1U" H 9675 9325 60  0001 C CNN
+F 2 "Alps_Only:ALPS-6.25U" H 9675 9325 60  0001 C CNN
 F 3 "" H 9675 9325 60  0001 C CNN
 	1    10300 9350
@@
 F 0 "MX-RWin2" H 12772 9295 60  0000 R CNN
 F 1 "MX-NoLED" H 12772 9369 20  0000 R CNN
-F 2 "Alps_Only:ALPS-1U" H 12275 9325 60  0001 C CNN
+F 2 "Alps_Only:ALPS-1.25U" H 12275 9325 60  0001 C CNN
 F 3 "" H 12275 9325 60  0001 C CNN
 	1    12900 9350
@@
 F 0 "MX-LAlt2" H 7572 9295 60  0000 R CNN
 F 1 "MX-NoLED" H 7572 9369 20  0000 R CNN
-F 2 "Alps_Only:ALPS-1U" H 7075 9325 60  0001 C CNN
+F 2 "Alps_Only:ALPS-1.25U" H 7075 9325 60  0001 C CNN
 F 3 "" H 7075 9325 60  0001 C CNN
 	1    7700 9350
@@
 F 0 "MX-LWin2" H 6922 9295 60  0000 R CNN
 F 1 "MX-NoLED" H 6922 9369 20  0000 R CNN
-F 2 "Alps_Only:ALPS-1U" H 6425 9325 60  0001 C CNN
+F 2 "Alps_Only:ALPS-1.25U" H 6425 9325 60  0001 C CNN
 F 3 "" H 6425 9325 60  0001 C CNN
 	1    7050 9350
@@
 F 0 "MX-LCtrl2" H 5622 9295 60  0000 R CNN
 F 1 "MX-NoLED" H 5622 9369 20  0000 R CNN
-F 2 "Alps_Only:ALPS-1U" H 5125 9325 60  0001 C CNN
+F 2 "Alps_Only:ALPS-1.25U" H 5125 9325 60  0001 C CNN
 F 3 "" H 5125 9325 60  0001 C CNN
 	1    5750 9350
@@
 F 0 "MX-Tab1" H 5783 6723 60  0000 C CNN
 F 1 "MX-NoLED" H 5783 6649 20  0000 C CNN
-F 2 "Alps_Only:ALPS-1U" H 5125 6475 60  0001 C CNN
+F 2 "Alps_Only:ALPS-1.5U" H 5125 6475 60  0001 C CNN
 F 3 "" H 5125 6475 60  0001 C CNN
 	1    5750 6500
@@
 	12850 8900 12850 9500
 Connection ~ 12850 8900
+Text Label 10000 1800 0    50   ~ 0
+D-
+Text Label 10000 1900 0    50   ~ 0
+D+
+Text Label 1750 2600 0    50   ~ 0
+D+
+Text Label 950  2600 0    50   ~ 0
+D+
+Text Label 1700 2700 0    50   ~ 0
+D-
+Text Label 900  2700 0    50   ~ 0
+D-
 $EndSCHEMATC

Commit message: Schematic update
Parts:
- MX-Esc1, MX-Fn1, MX-LWin1, MX-PgDn1, MX-PgUp1, MX-Super1: footprint Alps_Only:ALPS-1U -> MX_Alps_Hybrid:MX-1U-NoLED
Changed lines of the file:
@@
 F 0 "MX-Esc1" H 5783 5973 60  0000 C CNN
 F 1 "MX-NoLED" H 5783 5899 20  0000 C CNN
-F 2 "Alps_Only:ALPS-1U" H 5125 5725 60  0001 C CNN
+F 2 "MX_Alps_Hybrid:MX-1U-NoLED" H 5125 5725 60  0001 C CNN
 F 3 "" H 5125 5725 60  0001 C CNN
 	1    5750 5750
@@
 F 0 "MX-PgUp1" H 15533 5973 60  0000 C CNN
 F 1 "MX-NoLED" H 15533 5899 20  0000 C CNN
-F 2 "Alps_Only:ALPS-1U" H 14875 5725 60  0001 C CNN
+F 2 "MX_Alps_Hybrid:MX-1U-NoLED" H 14875 5725 60  0001 C CNN
 F 3 "" H 14875 5725 60  0001 C CNN
 	1    15500 5750
@@
 F 0 "MX-PgDn1" H 15533 6723 60  0000 C CNN
 F 1 "MX-NoLED" H 15533 6649 20  0000 C CNN
-F 2 "Alps_Only:ALPS-1U" H 14875 6475 60  0001 C CNN
+F 2 "MX_Alps_Hybrid:MX-1U-NoLED" H 14875 6475 60  0001 C CNN
 F 3 "" H 14875 6475 60  0001 C CNN
 	1    15500 6500
@@
 F 0 "MX-Super1" H 15533 7473 60  0000 C CNN
 F 1 "MX-NoLED" H 15533 7399 20  0000 C CNN
-F 2 "Alps_Only:ALPS-1U" H 14875 7225 60  0001 C CNN
+F 2 "MX_Alps_Hybrid:MX-1U-NoLED" H 14875 7225 60  0001 C CNN
 F 3 "" H 14875 7225 60  0001 C CNN
 	1    15500 7250
@@
 F 0 "MX-Fn1" H 15533 8223 60  0000 C CNN
 F 1 "MX-NoLED" H 15533 8149 20  0000 C CNN
-F 2 "Alps_Only:ALPS-1U" H 14875 7975 60  0001 C CNN
+F 2 "MX_Alps_Hybrid:MX-1U-NoLED" H 14875 7975 60  0001 C CNN
 F 3 "" H 14875 7975 60  0001 C CNN
 	1    15500 8000
@@
 F 0 "MX-LWin1" H 7083 8973 60  0000 C CNN
 F 1 "MX-NoLED" H 7083 8899 20  0000 C CNN
-F 2 "Alps_Only:ALPS-1U" H 6425 8725 60  0001 C CNN
+F 2 "MX_Alps_Hybrid:MX-1U-NoLED" H 6425 8725 60  0001 C CNN
 F 3 "" H 6425 8725 60  0001 C CNN
 	1    7050 8750

Commit message: PCB update
Parts:
- U1: footprint Package_QFP:TQFP-44_10x10mm_P0.8mm -> Housings_QFP:TQFP-44_10x10mm_Pitch0.8mm
Changed lines of the file:
@@
 F 0 "U1" H 2600 1211 50  0000 C CNN
 F 1 "ATmega32U4-AU" H 2600 1120 50  0000 C CNN
-F 2 "Package_QFP:TQFP-44_10x10mm_P0.8mm" H 2600 3100 50  0001 C CIN
+F 2 "Housings_QFP:TQFP-44_10x10mm_Pitch0.8mm" H 2600 3100 50  0001 C CIN
 F 3 "http://ww1.microchip.com/downloads/en/DeviceDoc/Atmel-7766-8-bit-AVR-ATmega16U4-32U4_Datasheet.pdf" H 2600 3100 50  0001 C CNN
 	1    2600 3100

Commit message: Update Schematic
Parts:
- MX-RWin1: footprint Alps_Only:ALPS-1U -> Alps_Only:ALPS-1.5U
Connections:
- net COL0: now also MX-LCtrl2.2 (ROW); no longer MX-LCtrl2.1 (COL)
- net COL11: now also MX-RWin2.2 (ROW); no longer MX-RWin2.1 (COL)
- net COL14: now also MX-Backspace2.1 (COL); no longer MX-Backspace2.2 (ROW)
- net COL2: now also MX-LWin2.2 (ROW); no longer MX-LWin2.1 (COL)
- net COL3: now also MX-LAlt2.2 (ROW); no longer MX-LAlt2.1 (COL)
- net at D15.2 (A), MX-Backspace1.2 (ROW): now also MX-Backspace2.2 (ROW); no longer MX-Backspace2.1 (COL)
- net at D60.2 (A), MX-LCtrl1.2 (ROW): now also MX-LCtrl2.1 (COL); no longer MX-LCtrl2.2 (ROW)
- net at D61.2 (A), MX-LWin1.2 (ROW): now also MX-LWin2.1 (COL); no longer MX-LWin2.2 (ROW)
- net at D62.2 (A), MX-LAlt1.2 (ROW): now also MX-LAlt2.1 (COL); no longer MX-LAlt2.2 (ROW)
- net at D65.2 (A), MX-RWin1.2 (ROW): now also MX-RWin2.1 (COL); no longer MX-RWin2.2 (ROW)
Other:
- moved on the sheet: MX-Backspace2, MX-LAlt2, MX-LCtrl2, MX-LWin2, MX-RWin2
Changed lines of the file:
@@
 	13950 5900 14150 5900
-$Comp
-L MX_Alps_Hybrid:MX-NoLED MX-Backspace1
-U 1 1 5DFC326B
-P 14850 5750
-F 0 "MX-Backspace1" H 14883 5973 60  0000 C CNN
-F 1 "MX-NoLED" H 14883 5899 20  0000 C CNN
-F 2 "Alps_Only:ALPS-1U" H 14225 5725 60  0001 C CNN
-F 3 "" H 14225 5725 60  0001 C CNN
-	1    14850 5750
-	1    0    0    -1
-$EndComp
 $Comp
 L Device:D_Small D15
@@
 	12000 8900 12200 8900
 $Comp
-L MX_Alps_Hybrid:MX-NoLED MX-RWin1
-U 1 1 5E258093
-P 12900 8750
-F 0 "MX-RWin1" H 12933 8973 60  0000 C CNN
-F 1 "MX-NoLED" H 12933 8899 20  0000 C CNN
-F 2 "Alps_Only:ALPS-1U" H 12275 8725 60  0001 C CNN
-F 3 "" H 12275 8725 60  0001 C CNN
-	1    12900 8750
-	1    0    0    -1
-$EndComp
-$Comp
 L Device:D_Small D65
 U 1 1 5E258099
@@
 Wire Wire Line
 	14350 7950 14350 8700
-Wire Wire Line
-	15000 5250 15000 5700
-Connection ~ 15000 5700
-Wire Wire Line
-	15000 5700 15000 6450
 Connection ~ 15000 6450
 Wire Wire Line
@@
 L MX_Alps_Hybrid:MX-NoLED MX-Backspace2
 U 1 1 5E470851
-P 14650 5350
-F 0 "MX-Backspace2" H 14683 5573 60  0000 C CNN
-F 1 "MX-NoLED" H 14683 5499 20  0000 C CNN
-F 2 "Alps_Only:ALPS-2U" H 14025 5325 60  0001 C CNN
-F 3 "" H 14025 5325 60  0001 C CNN
-	1    14650 5350
-	0    -1   -1   0
-$EndComp
-Wire Wire Line
-	14800 5400 14800 5700
-Wire Wire Line
-	14800 5700 15000 5700
-Wire Wire Line
-	14600 5200 14600 5900
-Connection ~ 14600 5900
+P 14650 5550
+F 0 "MX-Backspace2" H 14683 5773 60  0000 C CNN
+F 1 "MX-NoLED" H 14683 5699 20  0000 C CNN
+F 2 "Alps_Only:ALPS-2U" H 14025 5525 60  0001 C CNN
+F 3 "" H 14025 5525 60  0001 C CNN
+	1    14650 5550
+	1    0    0    -1
+$EndComp
 $Comp
 L MX_Alps_Hybrid:MX-NoLED MX-Space2
@@
 F 3 "" H 12275 9325 60  0001 C CNN
 	1    12900 9350
-	1    0    0    -1
+	0    -1   -1   0
 $EndComp
 $Comp
@@
 F 3 "" H 7075 9325 60  0001 C CNN
 	1    7700 9350
-	1    0    0    -1
-$EndComp
-$Comp
-L MX_Alps_Hybrid:MX-NoLED MX-LWin2
-U 1 1 5E552419
-P 7050 9350
-F 0 "MX-LWin2" H 6922 9295 60  0000 R CNN
-F 1 "MX-NoLED" H 6922 9369 20  0000 R CNN
-F 2 "Alps_Only:ALPS-1.25U" H 6425 9325 60  0001 C CNN
-F 3 "" H 6425 9325 60  0001 C CNN
-	1    7050 9350
-	1    0    0    -1
+	0    -1   -1   0
 $EndComp
 $Comp
@@
 F 3 "" H 5125 9325 60  0001 C CNN
 	1    5750 9350
-	1    0    0    -1
+	0    -1   -1   0
 $EndComp
 Text GLabel 5200 6100 0    50   Input ~ 0
@@
 	10250 8900 10250 9500
 Connection ~ 10250 8900
-Wire Wire Line
-	7850 8700 7850 9300
-Connection ~ 7850 8700
-Wire Wire Line
-	7650 8900 7650 9500
-Connection ~ 7650 8900
-Wire Wire Line
-	7200 8700 7200 9300
-Connection ~ 7200 8700
-Wire Wire Line
-	7000 8900 7000 9500
-Connection ~ 7000 8900
-Wire Wire Line
-	5900 8700 5900 9300
-Connection ~ 5900 8700
-Wire Wire Line
-	5700 8900 5700 9500
-Connection ~ 5700 8900
-Wire Wire Line
-	13050 8700 13050 9300
-Connection ~ 13050 8700
-Wire Wire Line
-	12850 8900 12850 9500
-Connection ~ 12850 8900
 Text Label 10000 1800 0    50   ~ 0
 D-
@@
 Text Label 900  2700 0    50   ~ 0
 D-
+Wire Wire Line
+	5900 8700 5900 9400
+Connection ~ 5900 8700
+Wire Wire Line
+	5700 9200 5700 8900
+Connection ~ 5700 8900
+$Comp
+L MX_Alps_Hybrid:MX-NoLED MX-LWin2
+U 1 1 5E552419
+P 7050 9350
+F 0 "MX-LWin2" H 6922 9295 60  0000 R CNN
+F 1 "MX-NoLED" H 6922 9369 20  0000 R CNN
+F 2 "Alps_Only:ALPS-1.25U" H 6425 9325 60  0001 C CNN
+F 3 "" H 6425 9325 60  0001 C CNN
+	1    7050 9350
+	0    -1   -1   0
+$EndComp
+Wire Wire Line
+	7000 8900 7000 9200
+Connection ~ 7000 8900
+Wire Wire Line
+	7200 8700 7200 9400
+Connection ~ 7200 8700
+Wire Wire Line
+	7650 8900 7650 9200
+Connection ~ 7650 8900
+Wire Wire Line
+	7850 8700 7850 9400
+Connection ~ 7850 8700
+$Comp
+L MX_Alps_Hybrid:MX-NoLED MX-RWin1
+U 1 1 5E258093
+P 12900 8750
+F 0 "MX-RWin1" H 12933 8973 60  0000 C CNN
+F 1 "MX-NoLED" H 12933 8899 20  0000 C CNN
+F 2 "Alps_Only:ALPS-1.5U" H 12275 8725 60  0001 C CNN
+F 3 "" H 12275 8725 60  0001 C CNN
+	1    12900 8750
+	1    0    0    -1
+$EndComp
+Wire Wire Line
+	12850 8900 12850 9200
+Connection ~ 12850 8900
+Wire Wire Line
+	13050 8700 13050 9400
+Connection ~ 13050 8700
+$Comp
+L MX_Alps_Hybrid:MX-NoLED MX-Backspace1
+U 1 1 5DFC326B
+P 14850 5750
+F 0 "MX-Backspace1" H 14883 5973 60  0000 C CNN
+F 1 "MX-NoLED" H 14883 5899 20  0000 C CNN
+F 2 "Alps_Only:ALPS-1U" H 14225 5725 60  0001 C CNN
+F 3 "" H 14225 5725 60  0001 C CNN
+	1    14850 5750
+	1    0    0    -1
+$EndComp
+Wire Wire Line
+	15000 5250 15000 5700
+Connection ~ 15000 5700
+Wire Wire Line
+	15000 5700 15000 6450
+Wire Wire Line
+	14800 5500 14800 5700
+Wire Wire Line
+	14800 5700 15000 5700
+Wire Wire Line
+	14600 5700 14600 5900
+Connection ~ 14600 5900
 $EndSCHEMATC

Commit message: PCB Update
Connections:
- net MOSI is gone; now on net COL1: J2.4 (MOSI), U1.10 (PB2)
- net SCK is gone; now on net COL0: J2.3 (SCK), U1.9 (PB1)
- net COL10: now also U1.38 (PF5)
- net COL11: now also U1.39 (PF4)
- net COL12: now also U1.21 (PD3)
- net COL13: now also U1.40 (PF1)
- net COL14: now also U1.25 (PD4)
- net COL15: now also U1.22 (PD5)
- net COL2: now also U1.31 (PC6)
- net COL3: now also U1.36 (PF7)
- net COL4: now also U1.30 (PB6)
- net COL5: now also U1.29 (PB5)
- net COL6: now also U1.28 (PB4)
- net COL7: now also U1.37 (PF6)
- net COL8: now also U1.27 (PD7)
- net COL9: now also U1.26 (PD6)
- net ROW0: now also U1.19 (PD1)
- net ROW1: now also U1.20 (PD2)
- net ROW2: now also U1.18 (PD0)
- net ROW3: now also U1.8 (PB0)
- net ROW4: now also U1.41 (PF0)
Changed lines of the file:
@@
 $EndDescr
-$Comp
-L MCU_Microchip_ATmega:ATmega32U4-AU U1
-U 1 1 5DF6F14B
-P 2600 3100
-F 0 "U1" H 2600 1211 50  0000 C CNN
-F 1 "ATmega32U4-AU" H 2600 1120 50  0000 C CNN
-F 2 "Housings_QFP:TQFP-44_10x10mm_Pitch0.8mm" H 2600 3100 50  0001 C CIN
-F 3 "http://ww1.microchip.com/downloads/en/DeviceDoc/Atmel-7766-8-bit-AVR-ATmega16U4-32U4_Datasheet.pdf" H 2600 3100 50  0001 C CNN
-	1    2600 3100
-	1    0    0    -1
-$EndComp
 $Comp
 L power:+5V #PWR0101
@@
 Wire Wire Line
 	1700 1600 1950 1600
-Text GLabel 3400 1900 2    50   Input ~ 0
+Text GLabel 3750 2000 2    50   Input ~ 0
 MISO
-Text GLabel 3400 1800 2    50   Input ~ 0
+Text GLabel 3750 1800 2    50   Input ~ 0
 MOSI
-Text GLabel 3400 1700 2    50   Input ~ 0
+Text GLabel 3750 1700 2    50   Input ~ 0
 SCK
-Wire Wire Line
-	3200 1700 3400 1700
-Wire Wire Line
-	3400 1800 3200 1800
-Wire Wire Line
-	3200 1900 3400 1900
 $Comp
 L Connector:AVR-ISP-6 J2
@@
 	14600 5700 14600 5900
 Connection ~ 14600 5900
+Text GLabel 3400 1600 2    50   Input ~ 0
+ROW3
+Wire Wire Line
+	3200 1600 3400 1600
+Text GLabel 3750 1600 2    50   Input ~ 0
+COL0
+Text GLabel 3750 1900 2    50   Input ~ 0
+COL1
+Text GLabel 3400 2500 2    50   Input ~ 0
+COL2
+Wire Wire Line
+	3700 1600 3700 1700
+Wire Wire Line
+	3700 1700 3200 1700
+Wire Wire Line
+	3700 1600 3750 1600
+Wire Wire Line
+	3700 1700 3750 1700
+Connection ~ 3700 1700
+Wire Wire Line
+	3200 1800 3700 1800
+Wire Wire Line
+	3700 1800 3700 1900
+Wire Wire Line
+	3700 1900 3750 1900
+Connection ~ 3700 1800
+Wire Wire Line
+	3700 1800 3750 1800
+Wire Wire Line
+	3650 1900 3650 2000
+Wire Wire Line
+	3200 1900 3650 1900
+Text GLabel 3400 2900 2    50   Input ~ 0
+ROW0
+Text GLabel 3400 3000 2    50   Input ~ 0
+ROW1
+Text GLabel 3400 2800 2    50   Input ~ 0
+ROW2
+Wire Wire Line
+	3200 2800 3400 2800
+Wire Wire Line
+	3200 2900 3400 2900
+Wire Wire Line
+	3200 3000 3400 3000
+Text GLabel 3400 4000 2    50   Input ~ 0
+ROW4
+Wire Wire Line
+	3400 4000 3200 4000
+Text GLabel 3400 4400 2    50   Input ~ 0
+COL7
+Text GLabel 3400 4300 2    50   Input ~ 0
+COL10
+Text GLabel 3400 4200 2    50   Input ~ 0
+COL11
+Text GLabel 3400 4100 2    50   Input ~ 0
+COL13
+Text GLabel 3400 4500 2    50   Input ~ 0
+COL3
+Wire Wire Line
+	3200 4100 3400 4100
+Wire Wire Line
+	3200 4200 3400 4200
+Wire Wire Line
+	3200 4300 3400 4300
+Wire Wire Line
+	3200 4400 3400 4400
+Wire Wire Line
+	3200 4500 3400 4500
+Text GLabel 3750 2400 2    50   Input ~ 0
+COL4
+Text GLabel 3750 2300 2    50   Input ~ 0
+COL5
+Text GLabel 3750 2200 2    50   Input ~ 0
+COL6
+Text GLabel 3400 3500 2    50   Input ~ 0
+COL8
+Text GLabel 3400 3400 2    50   Input ~ 0
+COL9
+Text GLabel 3400 3100 2    50   Input ~ 0
+COL12
+Text GLabel 3400 3200 2    50   Input ~ 0
+COL14
+Text GLabel 3400 3300 2    50   Input ~ 0
+COL15
+Wire Wire Line
+	3200 2000 3600 2000
+Wire Wire Line
+	3600 2000 3600 2200
+Wire Wire Line
+	3600 2200 3750 2200
+Wire Wire Line
+	3200 2100 3550 2100
+Wire Wire Line
+	3550 2100 3550 2300
+Wire Wire Line
+	3550 2300 3750 2300
+Wire Wire Line
+	3200 2200 3500 2200
+Wire Wire Line
+	3500 2200 3500 2400
+Wire Wire Line
+	3500 2400 3750 2400
+Wire Wire Line
+	3200 3100 3400 3100
+Wire Wire Line
+	3400 3200 3200 3200
+Wire Wire Line
+	3200 3300 3400 3300
+Wire Wire Line
+	3400 3400 3200 3400
+Wire Wire Line
+	3200 3500 3400 3500
+$Comp
+L MCU_Microchip_ATmega:ATmega32U4-AU U1
+U 1 1 5DF6F14B
+P 2600 3100
+F 0 "U1" H 2600 1211 50  0000 C CNN
+F 1 "ATmega32U4-AU" H 2600 1120 50  0000 C CNN
+F 2 "Housings_QFP:TQFP-44_10x10mm_Pitch0.8mm" H 2600 3100 50  0001 C CIN
+F 3 "http://ww1.microchip.com/downloads/en/DeviceDoc/Atmel-7766-8-bit-AVR-ATmega16U4-32U4_Datasheet.pdf" H 2600 3100 50  0001 C CNN
+	1    2600 3100
+	1    0    0    -1
+$EndComp
+Wire Wire Line
+	3200 2500 3400 2500
+Wire Wire Line
+	3650 2000 3750 2000
 $EndSCHEMATC

Commit message: PCB Update
Connections:
- net COL11: now also U1.37 (PF6); no longer U1.39 (PF4)
- net COL13: now also U1.36 (PF7); no longer U1.40 (PF1)
- net COL3: now also U1.40 (PF1); no longer U1.36 (PF7)
- net COL7: now also U1.39 (PF4); no longer U1.37 (PF6)
Changed lines of the file:
@@
 Wire Wire Line
 	3400 4000 3200 4000
-Text GLabel 3400 4400 2    50   Input ~ 0
+Text GLabel 3400 4200 2    50   Input ~ 0
 COL7
 Text GLabel 3400 4300 2    50   Input ~ 0
 COL10
-Text GLabel 3400 4200 2    50   Input ~ 0
+Text GLabel 3400 4400 2    50   Input ~ 0
 COL11
+Text GLabel 3400 4500 2    50   Input ~ 0
+COL13
 Text GLabel 3400 4100 2    50   Input ~ 0
-COL13
-Text GLabel 3400 4500 2    50   Input ~ 0
 COL3
 Wire Wire Line
