File: kc65alps.sch (KiCad schematic (older format))
At the start: 160 parts, among them J1 Conn_01x04, J2 AVR-ISP-6, U1 ATmega32U4-AU, Y1 16MHz

Commit message: PCB update
Connections:
- net ROW3: now also U1.32 (PC7); no longer U1.8 (PB0)
Changed lines of the file:
@@
 	14600 5700 14600 5900
 Connection ~ 14600 5900
-Text GLabel 3400 1600 2    50   Input ~ 0
+Text GLabel 3400 2600 2    50   Input ~ 0
 ROW3
-Wire Wire Line
-	3200 1600 3400 1600
 Text GLabel 3750 1600 2    50   Input ~ 0
 COL0
@@
 Wire Wire Line
 	3650 2000 3750 2000
+Wire Wire Line
+	3400 2600 3200 2600
 $EndSCHEMATC
