File: kc65alps.sch (KiCad schematic (older format))
At the start: 160 parts, among them J1 Conn_01x04, J2 AVR-ISP-6, U1 ATmega32U4-AU, Y1 16MHz

Commit message: PCB update
Parts:
- MX-Fn1, MX-LWin1, MX-PgDn1, MX-PgUp1, MX-Super1: footprint MX_Alps_Hybrid:MX-1U-NoLED -> Alps_Only:ALPS-1U
Changed lines of the file:
@@
 F 0 "MX-PgUp1" H 15533 5973 60  0000 C CNN
 F 1 "MX-NoLED" H 15533 5899 20  0000 C CNN
-F 2 "MX_Alps_Hybrid:MX-1U-NoLED" H 14875 5725 60  0001 C CNN
+F 2 "Alps_Only:ALPS-1U" H 14875 5725 60  0001 C CNN
 F 3 "" H 14875 5725 60  0001 C CNN
 	1    15500 5750
@@
 F 0 "MX-PgDn1" H 15533 6723 60  0000 C CNN
 F 1 "MX-NoLED" H 15533 6649 20  0000 C CNN
-F 2 "MX_Alps_Hybrid:MX-1U-NoLED" H 14875 6475 60  0001 C CNN
+F 2 "Alps_Only:ALPS-1U" H 14875 6475 60  0001 C CNN
 F 3 "" H 14875 6475 60  0001 C CNN
 	1    15500 6500
@@
 F 0 "MX-Super1" H 15533 7473 60  0000 C CNN
 F 1 "MX-NoLED" H 15533 7399 20  0000 C CNN
-F 2 "MX_Alps_Hybrid:MX-1U-NoLED" H 14875 7225 60  0001 C CNN
+F 2 "Alps_Only:ALPS-1U" H 14875 7225 60  0001 C CNN
 F 3 "" H 14875 7225 60  0001 C CNN
 	1    15500 7250
@@
 F 0 "MX-Fn1" H 15533 8223 60  0000 C CNN
 F 1 "MX-NoLED" H 15533 8149 20  0000 C CNN
-F 2 "MX_Alps_Hybrid:MX-1U-NoLED" H 14875 7975 60  0001 C CNN
+F 2 "Alps_Only:ALPS-1U" H 14875 7975 60  0001 C CNN
 F 3 "" H 14875 7975 60  0001 C CNN
 	1    15500 8000
@@
 F 0 "MX-LWin1" H 7083 8973 60  0000 C CNN
 F 1 "MX-NoLED" H 7083 8899 20  0000 C CNN
-F 2 "MX_Alps_Hybrid:MX-1U-NoLED" H 6425 8725 60  0001 C CNN
+F 2 "Alps_Only:ALPS-1U" H 6425 8725 60  0001 C CNN
 F 3 "" H 6425 8725 60  0001 C CNN
 	1    7050 8750
