File: kc65alps.kicad_pcb (KiCad board)
At the start: 2 copper layers, 160 parts, among them J1 Conn_01x04, J2 AVR-ISP-6, U1 ATmega32U4-AU, Y1 16MHz

Commit message: PCB update
Parts:
- moved MX-Caps3 246.4 mm to (31.0, 127.0), turned to 180 degrees
- moved MX-Caps2 239.0 mm to (28.6, 127.0)
- moved MX-Caps1 233.7 mm to (33.3, 127.0)
Changed lines of the file:
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@@
     (solder_mask_min_width 0.25)
     (aux_axis_origin 0 0)
-    (visible_elements FFFFFF7F)
+    (visible_elements 7FFFF7FF)
     (pcbplotparams
       (layerselection 0x010fc_ffffffff)
@@
   )
   (module Alps_Only:ALPS-1U (layer F.Cu)
-    (at 131.7075 351.865)
+    (at 30.95625 127 180)
     (fp_text reference MX-Caps3 (at 0 3.175) (layer Dwgs.User)
       (effects (font (size 1 1) (thickness 0.15)))
@@
     (fp_line (start 7 -7) (end 7 -5) (layer Dwgs.User) (width 0.15))
     (fp_line (start 5 -7) (end 7 -7) (layer Dwgs.User) (width 0.15))
-    (pad 1 thru_hole circle (at -2.5 -4) (size 2.25 2.25) (drill 1.47) (layers *.Cu B.Mask)
+    (pad 1 thru_hole circle (at -2.5 -4 180) (size 2.25 2.25) (drill 1.47) (layers *.Cu B.Mask)
       (net 40 "Net-(D32-Pad2)"))
-    (pad 2 thru_hole circle (at 2.5 -4.5) (size 2.25 2.25) (drill 1.47) (layers *.Cu B.Mask)
+    (pad 2 thru_hole circle (at 2.5 -4.5 180) (size 2.25 2.25) (drill 1.47) (layers *.Cu B.Mask)
       (net 100 COL0))
   )
   (module Alps_Only:ALPS-1U (layer F.Cu)
-    (at 151.9075 331.665)
+    (at 28.575 127)
     (fp_text reference MX-Caps2 (at 0 3.175) (layer Dwgs.User)
       (effects (font (size 1 1) (thickness 0.15)))
@@
   )
   (module Alps_Only:ALPS-1U (layer F.Cu)
-    (at 176.8675 311.465)
+    (at 33.3375 127)
     (fp_text reference MX-Caps1 (at 0 3.175) (layer Dwgs.User)
       (effects (font (size 1 1) (thickness 0.15)))

Commit message: PCB update
Parts:
- moved MX-Caps1 2.38 mm to (35.7, 127.0)
- moved MX-Caps2 2.38 mm to (31.0, 127.0)
- moved MX-Caps3 2.38 mm to (33.3, 127.0)
Changed lines of the file:
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@@
   )
   (module Alps_Only:ALPS-1U (layer F.Cu)
-    (at 30.95625 127 180)
+    (at 33.3375 127 180)
     (fp_text reference MX-Caps3 (at 0 3.175) (layer Dwgs.User)
       (effects (font (size 1 1) (thickness 0.15)))
@@
   )
   (module Alps_Only:ALPS-1U (layer F.Cu)
-    (at 28.575 127)
+    (at 30.95625 127)
     (fp_text reference MX-Caps2 (at 0 3.175) (layer Dwgs.User)
       (effects (font (size 1 1) (thickness 0.15)))
@@
   )
   (module Alps_Only:ALPS-1U (layer F.Cu)
-    (at 33.3375 127)
+    (at 35.71875 127)
     (fp_text reference MX-Caps1 (at 0 3.175) (layer Dwgs.User)
       (effects (font (size 1 1) (thickness 0.15)))

Commit message: PCB update
Parts:
- D1, D10, D11, D12, D13, D14, D15, D16, D17, D18, D19, D2, D20, D21, D22, D23, D24, D25, D26, D27, D28, D29, D3, D30, D31, D32, D33, D34, D35, D36, D37, D38, D39, D4, D40, D41, D42, D43, D44, D45, D46, D47, D48, D49, D5, D50, D51, D52, D53, D54, D55, D56, D57, D58, D59, D6, D60, D61, D62, D63, D64, D65, D66, D67, D68, D7, D8, D9, J1, R2, R3, U1: moved to B.Cu
- moved D68 354.6 mm to (321.5, 162.7), turned to 90 degrees
- moved D67 335.1 mm to (303.2, 162.7), turned to 90 degrees
- moved D11 319.6 mm to (228.6, 86.5), turned to 90 degrees
- moved D66 316.9 mm to (285.8, 162.7), turned to 90 degrees
- moved D59 315.0 mm to (306.4, 143.7), turned to 90 degrees
- moved D13 314.9 mm to (265.1, 86.5), turned to 90 degrees
- moved D58 308.6 mm to (303.2, 143.7), turned to 90 degrees
- moved D16 305.1 mm to (306.4, 86.5), turned to 90 degrees
- moved D12 304.6 mm to (247.7, 86.5), turned to 90 degrees
- moved D1 301.0 mm to (38.1, 86.5), turned to 90 degrees
- moved D17 295.5 mm to (42.9, 105.6), turned to 90 degrees
- moved D57 288.1 mm to (278.6, 143.7), turned to 90 degrees
- moved D65 287.7 mm to (252.4, 162.7), turned to 90 degrees
- moved D2 287.2 mm to (57.1, 86.5), turned to 90 degrees
- moved R2 284.8 mm to (24.1, 121.9), turned to 90 degrees
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Other:
- board outline added: 304.8 x 95.3 mm

Commit message: PCB update
Parts:
- C1, C2, C3, C4, C5, C6, C7, F1, R1, R4, Y1: moved to B.Cu
- moved C3 266.2 mm to (46.1, 143.3), turned to 180 degrees
- moved C2 260.2 mm to (51.6, 132.7), turned to 270 degrees
- moved C1 259.8 mm to (55.2, 129.4), turned to 180 degrees
- moved R1 259.6 mm to (44.5, 136.1), turned to 270 degrees
- moved C6 256.6 mm to (63.6, 136.7), turned to 90 degrees
- moved C5 255.9 mm to (47.8, 136.1), turned to 90 degrees
- moved Y1 255.1 mm to (55.2, 132.7), turned to 180 degrees
- moved C4 245.5 mm to (63.6, 150.1), turned to 270 degrees
- moved F1 150.6 mm to (25.4, 127.8), turned to 270 degrees
- moved C7 119.8 mm to (51.4, 151.3)
- moved J2 109.5 mm to (42.1, 153.2), turned to 90 degrees
- moved R4 101.1 mm to (65.7, 150.1), turned to 90 degrees
- moved U1 63.3 mm to (56.0, 143.1)
- moved D46 17.5 mm to (32.5, 143.7)
- moved D68 15.1 mm to (306.4, 162.7)
Connections:
- J2 pad 1: MISO -> COL2
- J2 pad 3: SCK -> COL0
- J2 pad 4: MOSI -> COL1
- U1 pad 10: MOSI -> COL1
- U1 pad 11: MISO -> COL2
- U1 pad 8: Net-(U1-Pad8) -> ROW3
- U1 pad 9: SCK -> COL0
Routing:
- net ROW3: track 0.00 -> 324.2 mm, vias 0 -> 2
- net ROW0: track 0.00 -> 268.3 mm
- net ROW4: track 0.00 -> 266.1 mm
- net ROW2: track 0.00 -> 263.5 mm
- net ROW1: track 0.00 -> 263.5 mm
- net COL2: track 0.00 -> 151.3 mm, vias 0 -> 1
- net GND: track 0.00 -> 127.3 mm
- net COL0: track 0.00 -> 120.3 mm, vias 0 -> 1
- net +5V: track 0.00 -> 118.7 mm, vias 0 -> 6
- net COL7: track 0.00 -> 100.9 mm
- net COL3: track 0.00 -> 99.5 mm
- net COL13: track 0.00 -> 95.9 mm
- net COL11: track 0.00 -> 95.5 mm
- net COL14: track 0.00 -> 90.6 mm
- net COL10: track 0.00 -> 87.0 mm
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Other:
- net class Default: trace_width 0.25 -> 0.254
- net class Power added: clearance 0.2, trace_width 0.381, via_dia 0.8, via_drill 0.4

Commit message: PCB Update
Connections:
- J2 pad 1: COL2 -> MISO
- U1 pad 11: COL2 -> MISO
- U1 pad 18: Net-(U1-Pad18) -> ROW2
- U1 pad 19: Net-(U1-Pad19) -> ROW0
- U1 pad 20: Net-(U1-Pad20) -> ROW1
- U1 pad 21: Net-(U1-Pad21) -> COL12
- U1 pad 22: Net-(U1-Pad22) -> COL15
- U1 pad 25: Net-(U1-Pad25) -> COL14
- U1 pad 26: Net-(U1-Pad26) -> COL9
- U1 pad 27: Net-(U1-Pad27) -> COL8
- U1 pad 28: Net-(U1-Pad28) -> COL6
- U1 pad 29: Net-(U1-Pad29) -> COL5
- U1 pad 30: Net-(U1-Pad30) -> COL4
- U1 pad 31: Net-(U1-Pad31) -> COL2
- U1 pad 36: Net-(U1-Pad36) -> COL3
- U1 pad 37: Net-(U1-Pad37) -> COL7
- U1 pad 38: Net-(U1-Pad38) -> COL10
- U1 pad 39: Net-(U1-Pad39) -> COL11
- U1 pad 40: Net-(U1-Pad40) -> COL13
- U1 pad 41: Net-(U1-Pad41) -> ROW4
Routing:
- net COL15: track 75.3 -> 332.2 mm
- net COL14: track 90.6 -> 324.6 mm
- net COL13: track 95.9 -> 310.2 mm, vias 0 -> 1
- net COL12: track 44.0 -> 251.3 mm, vias 0 -> 1
- net COL11: track 95.5 -> 282.6 mm, vias 0 -> 1
- net COL10: track 87.0 -> 254.2 mm, vias 0 -> 1
- net COL9: track 67.0 -> 210.5 mm
- net COL8: track 67.0 -> 191.4 mm
- net COL7: track 100.9 -> 209.8 mm, vias 0 -> 1
- net COL6: track 67.0 -> 153.2 mm
- net COL5: track 67.0 -> 134.1 mm
- net ROW0: track 268.3 -> 333.6 mm, vias 0 -> 2
- net COL4: track 67.0 -> 115.0 mm
- net ROW1: track 263.5 -> 310.1 mm, vias 0 -> 2
- net COL2: track 151.3 -> 110.2 mm, vias 1 -> 0
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
Commit message: PCB Update
Connections:
- U1 pad 36: COL3 -> COL13
- U1 pad 37: COL7 -> COL11
- U1 pad 39: COL11 -> COL7
- U1 pad 40: COL13 -> COL3
Routing:
- net COL7: track 209.8 -> 198.0 mm, vias 1 -> 0
- net COL13: track 310.2 -> 316.9 mm, vias 1 -> 0
- net COL3: track 130.8 -> 128.3 mm, vias 1 -> 0
- net COL11: track 282.6 -> 284.0 mm, vias 1 -> 0
- net COL10: track 254.2 -> 254.9 mm, vias 1 -> 0

Commit message: PCB update
Routing:
- added copper zone on B.Cu, net GND
Changed lines of the file:
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@@
   (segment (start 21.51875 119.075) (end 21.51875 119.55) (width 0.381) (layer B.Cu) (net 79))
   (segment (start 25.4 124.090357) (end 25.4 126.59375) (width 0.381) (layer B.Cu) (net 79))
-  (segment (start 21.51875 117.919) (end 21.528251 117.909499) (width 0.381) (layer B.Cu) (net 79))
-  (segment (start 21.51875 119.075) (end 21.51875 117.919) (width 0.381) (layer B.Cu) (net 79))
-  (segment (start 21.528251 117.909499) (end 25.131151 117.909499) (width 0.381) (layer B.Cu) (net 79))
+  (segment (start 21.51875 119.075) (end 21.51875 118.297098) (width 0.381) (layer B.Cu) (net 79))
+  (segment (start 21.906349 117.909499) (end 25.131151 117.909499) (width 0.381) (layer B.Cu) (net 79))
+  (segment (start 21.51875 118.297098) (end 21.906349 117.909499) (width 0.381) (layer B.Cu) (net 79))
   (segment (start 25.131151 117.909499) (end 25.751511 118.529859) (width 0.381) (layer B.Cu) (net 79))
   (segment (start 25.751511 118.529859) (end 25.751511 123.738846) (width 0.381) (layer B.Cu) (net 79))
@@
   (segment (start 64.1645 147.0655) (end 65.659 148.56) (width 0.254) (layer B.Cu) (net 100))
   (segment (start 61.707 147.0655) (end 64.1645 147.0655) (width 0.254) (layer B.Cu) (net 100))
+  (zone (net 2) (net_name GND) (layer B.Cu) (hatch edge 0.508)
+    (connect_pads (clearance 0.508))
+    (min_thickness 0.254)
+    (fill yes (arc_segments 32) (thermal_gap 0.508) (thermal_bridge_width 0.508))
+    (polygon
+      (pts
+        (xy 49.2125 136.525) (xy 62.70625 136.525) (xy 62.70625 150.01875) (xy 49.2125 150.01875)
+      )
+    )
+  )
+  (zone (net 2) (net_name GND) (layer B.Cu) (hatch edge 0.508)
+    (connect_pads (clearance 0.508))
+    (min_thickness 0.254)
+    (fill yes (arc_segments 32) (thermal_gap 0.508) (thermal_bridge_width 0.508))
+    (polygon
+      (pts
+        (xy 49.2125 134.14375) (xy 49.2125 126.20625) (xy 61.11875 126.20625) (xy 61.11875 134.14375)
+      )
+    )
+  )
 )

Commit message: PCB update
Parts:
- J2: moved to B.Cu
- moved F1 4.05 mm to (21.4, 127.0)
- moved D46 1.12 mm to (33.3, 142.9)
- moved J1 0.79 mm to (23.8, 114.3)
- moved R2 0.79 mm to (24.9, 121.9)
- moved R3 0.79 mm to (22.8, 121.9)
Routing:
- net +5V: track 118.7 -> 134.2 mm, vias 6 -> 5
- net RST: track 27.5 -> 37.1 mm
- net VCC: track 14.1 -> 7.09 mm
- net MISO: track 32.0 -> 26.2 mm
- net GND: track 127.3 -> 131.4 mm
- net D-: track 51.2 -> 49.9 mm
- net D+: track 50.5 -> 49.2 mm
- net Net-(D46-Pad2): track 11.6 -> 10.4 mm
