File: kc65alps.kicad_pcb (KiCad board)
At the start: 2 copper layers, 304.8 x 95.3 mm, 160 parts, among them J1 Conn_01x04, J2 AVR-ISP-6, U1 ATmega32U4-AU, Y1 16MHz

Commit message: PCB update
Parts:
- moved F1 18.8 mm to (25.3, 145.4), turned to 315 degrees
- moved C3 0.28 mm to (45.8, 143.1), turned to 270 degrees
Routing:
- net VCC: track 7.09 -> 27.1 mm
- net +5V: track 134.2 -> 116.9 mm
- net ROW4: track 286.9 -> 292.9 mm
- net COL15: track 332.2 -> 329.7 mm, vias 0 -> 1
- net Net-(D59-Pad2): track 11.4 -> 13.6 mm
- net Net-(D46-Pad2): track 10.4 -> 12.3 mm
- net Net-(C3-Pad1): track 3.28 -> 4.85 mm
- net Net-(C1-Pad1): track 9.07 -> 10.5 mm
- net MISO: track 26.2 -> 27.4 mm
- net Net-(D16-Pad2): track 11.5 -> 12.4 mm
- net Net-(D31-Pad2): track 11.5 -> 12.4 mm
- net Net-(D45-Pad2): track 11.4 -> 12.3 mm
- net GND: track 131.4 -> 132.0 mm
- net ROW3: track 324.2 -> 323.9 mm, vias 2 -> 3

Commit message: PCB update
Parts:
- MX-Fn1, MX-LWin1, MX-PgDn1, MX-PgUp1, MX-Super1: footprint MX_Alps_Hybrid:MX-1U-NoLED -> Alps_Only:ALPS-1U
- moved C1 0.89 mm to (55.2, 128.5)
- moved C2 0.89 mm to (51.6, 131.8)
- moved Y1 0.89 mm to (55.2, 131.8)
- moved C6 0.57 mm to (63.9, 137.2)
- moved C7 0.54 mm to (51.8, 151.6)
Connections:
- U1 pad 32: Net-(U1-Pad32) -> ROW3
- U1 pad 8: ROW3 -> Net-(U1-Pad8)
Routing:
- net +5V: track 116.9 -> 111.6 mm
- net COL15: track 329.7 -> 333.8 mm, vias 1 -> 0
- net ROW0: track 333.6 -> 329.8 mm
- net ROW1: track 310.1 -> 306.5 mm
- net COL12: track 251.3 -> 247.7 mm
- net GND: track 132.0 -> 135.1 mm, vias 0 -> 1
- net COL14: track 324.6 -> 327.2 mm
- net COL4: track 115.0 -> 117.2 mm
- net COL5: track 134.1 -> 136.3 mm
- net COL6: track 153.2 -> 155.3 mm
- net COL8: track 191.4 -> 193.5 mm
- net COL9: track 210.5 -> 212.6 mm
- net RST: track 37.1 -> 38.5 mm
- net Net-(C1-Pad1): track 10.5 -> 11.9 mm
- net ROW3: track 323.9 -> 322.7 mm, vias 3 -> 2
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- removed copper zone on B.Cu, net GND

Commit message: PCB update
Routing:
- net +5V: track 111.6 -> 112.5 mm
Changed lines of the file:
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@@
     (thickness 1.6)
     (drawings 8)
-    (tracks 635)
+    (tracks 636)
     (zones 0)
     (modules 160)
@@
   (segment (start 30.226 150.368) (end 26.121528 146.263528) (width 0.381) (layer B.Cu) (net 5))
   (segment (start 48.514 150.368) (end 30.226 150.368) (width 0.381) (layer B.Cu) (net 5))
-  (segment (start 46.95825 151.92375) (end 48.514 150.368) (width 0.381) (layer B.Cu) (net 5))
-  (segment (start 44.60875 151.92375) (end 46.95825 151.92375) (width 0.381) (layer B.Cu) (net 5))
   (segment (start 52.676859 135.49949) (end 51.347642 135.49949) (width 0.381) (layer B.Cu) (net 5))
   (segment (start 53.607 137.3655) (end 53.607 136.429631) (width 0.381) (layer B.Cu) (net 5))
@@
   (segment (start 61.468 150.368) (end 64.135 147.701) (width 0.381) (layer F.Cu) (net 5))
   (segment (start 48.514 150.368) (end 61.468 150.368) (width 0.381) (layer F.Cu) (net 5))
+  (segment (start 47.523935 151.92375) (end 46.38675 151.92375) (width 0.381) (layer B.Cu) (net 5))
+  (segment (start 48.514 150.933685) (end 47.523935 151.92375) (width 0.381) (layer B.Cu) (net 5))
+  (segment (start 48.514 150.368) (end 48.514 150.933685) (width 0.381) (layer B.Cu) (net 5))
+  (segment (start 44.60875 151.92375) (end 46.38675 151.92375) (width 0.381) (layer B.Cu) (net 5))
+  (segment (start 46.38675 151.92375) (end 46.95825 151.92375) (width 0.381) (layer B.Cu) (net 5))
   (segment (start 38.1 88.16875) (end 57.15 88.16875) (width 0.254) (layer B.Cu) (net 6))
   (segment (start 57.15 88.16875) (end 58.004 88.16875) (width 0.254) (layer B.Cu) (net 6))
@@
   (segment (start 24.92375 123.845001) (end 24.92375 122.87) (width 0.2) (layer B.Cu) (net 81))
   (segment (start 50.307 144.6655) (end 49.181999 144.6655) (width 0.2) (layer B.Cu) (net 81))
-  (segment (start 42.196788 137.094) (end 39.926048 139.36474) (width 0.254) (layer B.Cu) (net 82))
-  (segment (start 44.45 137.094) (end 42.196788 137.094) (width 0.254) (layer B.Cu) (net 82))
   (via (at 35.71875 139.09175) (size 0.8) (drill 0.4) (layers F.Cu B.Cu) (net 82))
-  (segment (start 39.926048 139.36474) (end 35.99174 139.36474) (width 0.254) (layer B.Cu) (net 82))
-  (segment (start 35.99174 139.36474) (end 35.71875 139.09175) (width 0.254) (layer B.Cu) (net 82))
   (segment (start 35.71875 150.65375) (end 39.52875 154.46375) (width 0.254) (layer F.Cu) (net 82))
   (segment (start 35.71875 139.09175) (end 35.71875 150.65375) (width 0.254) (layer F.Cu) (net 82))
@@
   (segment (start 47.16625 138.90625) (end 48.10125 138.90625) (width 0.254) (layer B.Cu) (net 82))
   (segment (start 48.10125 138.90625) (end 48.41875 138.90625) (width 0.254) (layer B.Cu) (net 82))
+  (segment (start 41.851913 137.094) (end 43.246 137.094) (width 0.254) (layer B.Cu) (net 82))
+  (segment (start 39.854163 139.09175) (end 41.851913 137.094) (width 0.254) (layer B.Cu) (net 82))
+  (segment (start 35.71875 139.09175) (end 39.854163 139.09175) (width 0.254) (layer B.Cu) (net 82))
+  (segment (start 44.45 137.094) (end 43.246 137.094) (width 0.254) (layer B.Cu) (net 82))
   (via (at 42.256249 138.36475) (size 0.8) (drill 0.4) (layers F.Cu B.Cu) (net 83))
   (segment (start 42.427999 138.5365) (end 42.256249 138.36475) (width 0.254) (layer B.Cu) (net 83))
@@
   (segment (start 41.529249 88.495751) (end 41.529249 138.502001) (width 0.254) (layer F.Cu) (net 86))
   (segment (start 45.125 84.9) (end 41.529249 88.495751) (width 0.254) (layer F.Cu) (net 86))
-  (via (at 41.275 139.09175) (size 0.8) (drill 0.4) (layers F.Cu B.Cu) (net 86))
-  (segment (start 41.138625 139.228125) (end 41.275 139.09175) (width 0.254) (layer F.Cu) (net 86))
-  (segment (start 40.803125 139.228125) (end 41.138625 139.228125) (width 0.254) (layer F.Cu) (net 86))
   (segment (start 40.803125 139.228125) (end 39.106249 140.925001) (width 0.254) (layer F.Cu) (net 86))
   (segment (start 41.529249 138.502001) (end 40.803125 139.228125) (width 0.254) (layer F.Cu) (net 86))
   (segment (start 37.98125 147.83625) (end 37.98125 142.05) (width 0.254) (layer F.Cu) (net 86))
   (segment (start 42.06875 151.92375) (end 37.98125 147.83625) (width 0.254) (layer F.Cu) (net 86))
-  (segment (start 41.840685 139.09175) (end 41.275 139.09175) (width 0.254) (layer B.Cu) (net 86))
-  (segment (start 46.067618 139.091751) (end 41.840685 139.09175) (width 0.254) (layer B.Cu) (net 86))
+  (segment (start 41.275 139.09175) (end 40.930125 139.09175) (width 0.254) (layer B.Cu) (net 86))
+  (segment (start 46.067618 139.091751) (end 41.275 139.09175) (width 0.254) (layer B.Cu) (net 86))
   (segment (start 46.841367 139.8655) (end 46.067618 139.091751) (width 0.254) (layer B.Cu) (net 86))
+  (via (at 40.930125 139.09175) (size 0.8) (drill 0.4) (layers F.Cu B.Cu) (net 86))
   (segment (start 50.307 139.8655) (end 46.841367 139.8655) (width 0.254) (layer B.Cu) (net 86))
   (segment (start 54.65 94.425) (end 64.175 84.9) (width 0.254) (layer F.Cu) (net 87))

Commit message: PCB update
Parts:
- moved F1 9.64 mm to (34.1, 149.2), turned to 0 degrees
Routing:
- net ROW3: track 322.7 -> 291.3 mm, vias 2 -> 4
- net +5V: track 112.5 -> 97.6 mm
- net VCC: track 27.1 -> 36.8 mm
- net GND: track 135.1 -> 139.9 mm, vias 1 -> 2
- net Net-(R4-Pad2): track 6.02 -> 5.18 mm
- added copper zone on B.Cu, net GND
- added copper zone on F.Cu, net GND
