File: kc65alps.kicad_pcb (KiCad board)
At the start: 2 copper layers, 304.8 x 95.3 mm, 160 parts, among them J1 Conn_01x04, J2 AVR-ISP-6, U1 ATmega32U4-AU, Y1 16MHz

Commit message: PCB update
Parts:
- added G***: LOGO, Hamshet_modules:Alps_symbol_test, B.Cu at (196.1, 162.7)
- moved C3 0.63 mm to (46.4, 142.7)
Routing:
- net GND: track 139.9 -> 129.4 mm
- net ROW3: track 291.3 -> 283.2 mm, vias 4 -> 2
- net COL0: track 122.1 -> 127.8 mm, vias 1 -> 0
- net +5V: track 97.6 -> 102.2 mm
- net MISO: track 28.4 -> 31.9 mm
- net ROW0: track 329.8 -> 327.9 mm
- net Net-(D46-Pad2): track 12.3 -> 10.6 mm
- net ROW4: track 292.9 -> 291.3 mm
- net COL14: track 327.2 -> 328.6 mm
- net Net-(D63-Pad2): track 20.1 -> 21.4 mm
- net RST: track 38.3 -> 39.3 mm

Commit message: PCB update
Parts:
- removed the G*** at (196.1, 162.7)
- added G***: LOGO, Hamshet_modules:Owl_Cave_Symbol_0.5in, B.Cu at (192.1, 158.8)
- moved C6 1.09 mm to (64.5, 136.3), turned to 180 degrees
- moved R4 0.89 mm to (66.5, 150.1)
- renumbered U1 to Howdy
Routing:
- net ROW4: track 291.3 -> 284.0 mm
- net GND: track 129.4 -> 122.4 mm, vias 2 -> 68
- net +5V: track 102.2 -> 105.2 mm
- net Net-(R4-Pad2): track 5.18 -> 6.06 mm
- net D+: track 49.2 -> 50.0 mm
